File: 555newbadge.kicad_pcb (KiCad board)
At the start: 2 copper layers, 53.8 x 85.6 mm, 15 parts, among them Q1 2N3904, U2 ICM7555xP

Commit message: Add files via upload
Routing:
- added copper zone on B.Cu, net GND
- added copper zone on F.Cu, net GND
Changed lines of the file:
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@@
   (segment (start 158.75 122.79737) (end 158.75 124.968) (width 0.25) (layer "B.Cu") (net 10))
   (segment (start 178.562 102.98537) (end 158.75 122.79737) (width 0.25) (layer "B.Cu") (net 10))
+  (zone (net 1) (net_name "GND") (layer "F.Cu") (hatch edge 0.5)
+    (connect_pads (clearance 0.5))
+    (min_thickness 0.25) (filled_areas_thickness no)
+    (fill yes (thermal_gap 0.5) (thermal_bridge_width 0.5))
+    (polygon
+      (pts
+        (xy 126.746 127.254)
+        (xy 126.746 41.148)
+        (xy 181.102 41.148)
+        (xy 181.102 127.254)
+      )
+    )
+  )
+  (zone (net 1) (net_name "GND") (layer "B.Cu") (hatch edge 0.5)
+    (priority 1)
+    (connect_pads (clearance 0.5))
+    (min_thickness 0.25) (filled_areas_thickness no)
+    (fill yes (thermal_gap 0.5) (thermal_bridge_width 0.5))
+    (polygon
+      (pts
+        (xy 126.746 127.254)
+        (xy 126.746 41.148)
+        (xy 181.102 41.148)
+        (xy 181.102 127.254)
+      )
+    )
+  )
   (zone (net 0) (net_name "") (layer "F.SilkS") (hatch edge 0.5)
     (connect_pads (clearance 0.5))
     (min_thickness 0.25) (filled_areas_thickness no)
-    (fill (thermal_gap 0.5) (thermal_bridge_width 0.5))
+    (fill yes (thermal_gap 0.5) (thermal_bridge_width 0.5))
     (polygon
       (pts
